File: PCB/SunLeaf-Sense-2.4G/SunLeaf-Sense-2.4G.kicad_pcb (KiCad board)
At the start: 4 copper layers, 100 x 40 mm, 75 parts, among them M1 SCD30, M2 STM32WB5MMGH6TR, Q1 DMP3125L-7, Q2 DMP3125L-7, SW1 B3U-1000P, T1 0395121002, T2 B3B-PH-K-S(LF)(SN), T3 20021121-00010C4LF, T4 DX07S016JA1R1500, U1 BQ24210DQCT, U10 OPA388IDBVT, U11 SN74LV4051ARGYR, U2 LTC2941CDCB-1#TRMPBF, U3 AZ1117CR-3.3TRG1, U4 TCA9546APWR, U5 AS7341-DLGT, U6 TPIS1T1086_L5.5, U7 HDC1080DMBR, U8 USBLC6-2P6, U9 HDC1080DMBR

Commit message: KiCAD 8
Projected updated to KiCAD 8
Other:
- net class Default removed
